Commit message: name change

File: wallbot.urdf (robot description, URDF)
Before this commit: robot wallbot, 12 links, 11 joints
Links:
- removed link sensor_left
- removed link sensor_right
- added link sensor_left_can; visual cylinder length=0.013 radius=0.008
- added link sensor_right_can; visual cylinder length=0.013 radius=0.008
Joints:
- joint sensor_left_joint: child sensor_left -> sensor_left_can
- joint sensor_right_joint: child sensor_right -> sensor_right_can
